File: 1.Project.Files/Probe Card/KiCAD Files/2.Bottom Probe Card/BottomProbeCard.kicad_pcb (KiCad board)
At the start: 2 copper layers, 160 x 87.6 mm, 2 parts

Commit message: Added all base files
Parts:
- removed ? (x2): , 
Routing:
- net (no net): track 146.6 -> 0.00 mm
- removed copper zone on B.Cu, net (none)
Other:
- board size 160 x 87.6 mm -> 70 x 87.5 mm
- board text added: "75.000 [mm]"
- board text added: "87.550 [mm]"
