File: 1.Project.Files/Probe Card/KiCAD Files/3.Probe Card Set/ProbeCardFull.kicad_pcb (KiCad board)
At the start: 2 copper layers, 160 x 87.6 mm, 2 parts

Commit message: Added all base files
Parts:
- added G***: LOGO, LOGO, F.Cu at (194.0, 107.0)
Other:
- board text added: "75.000 [mm]"
- board text added: "87.550 [mm]"
- board text added: "Department of Physics February 2024 https://github.com/barajasalfredo13/ModuTherm-Wafer-Test-System"
