File: 2.Probe Card/KiCAD Files/3.Probe Card Set/ProbeCardFull.kicad_pcb (KiCad board)
At the start: 2 copper layers, 160 x 87.6 mm, 3 parts

Commit message: Updated Documentation
Other:
- board text added: "70.000 [mm]"
- board text removed: "75.000 [mm]"
Changed lines of the file:
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@@
 	)
 	(gr_text "87.550 [mm]"
-		(at 35 33.724987 0)
+		(at 36 36 0)
 		(layer "User.4")
 		(effects
@@
 		)
 	)
-	(gr_text "75.000 [mm]"
-		(at 110 126.274987 0)
+	(gr_text "70.000 [mm]"
+		(at 94 125 0)
 		(layer "User.4")
 		(effects
